File: VCU2.0/CAN.kicad_sch (KiCad schematic)
At the start: 25 parts, among them U401 MCP2551-I/SN, U402 MCP2515-I/ST, U403 ADS1015IDGST, X401 K3A160002010

Commit message: simple regen
Connections:
- net +3.3V: now also R401.2, R402.2, U402.20 (VDD)
- net +5V: no longer R401.2, R402.2, U402.20 (VDD)
Changed lines of the file:
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@@
 	)
 	(junction
-		(at 90.17 26.67)
-		(diameter 0)
-		(color 0 0 0 0)
-	)
-	(junction
 		(at 149.86 106.68)
 		(diameter 0)
@@
 	)
 	(junction
+		(at 90.17 26.67)
+		(diameter 0)
+		(color 0 0 0 0)
+	)
+	(junction
 		(at 161.29 106.68)
 		(diameter 0)
@@
 	(wire
 		(pts
-			(xy 87.63 26.67) (xy 90.17 26.67)
-		)
-		(stroke
-			(width 0)
-			(type default)
-		)
-	)
-	(wire
-		(pts
 			(xy 22.86 60.96) (xy 41.91 60.96)
 		)
@@
 	(wire
 		(pts
+			(xy 90.17 26.67) (xy 92.71 26.67)
+		)
+		(stroke
+			(width 0)
+			(type default)
+		)
+	)
+	(wire
+		(pts
 			(xy 38.1 104.14) (xy 38.1 109.22)
 		)
@@
 	(wire
 		(pts
-			(xy 90.17 26.67) (xy 92.71 26.67)
+			(xy 87.63 26.67) (xy 90.17 26.67)
 		)
 		(stroke
@@
 	)
 	(symbol
+		(lib_id "power:+3.3V")
+		(at 41.91 44.45 0)
+		(unit 1)
+		(exclude_from_sim no)
+		(in_bom yes)
+		(on_board yes)
+		(dnp no)
+		(fields_autoplaced yes)
+		(property "Reference" "#PWR0403"
+			(at 41.91 48.26 0)
+			(effects
+				(font
+					(size 1.27 1.27)
+				)
+				(hide yes)
+			)
+		)
+		(property "Value" "+3.3V"
+			(at 41.91 39.37 0)
+			(effects
+				(font
+					(size 1.27 1.27)
+				)
+			)
+		)
+		(property "Footprint" ""
+			(at 41.91 44.45 0)
+			(effects
+				(font
+					(size 1.27 1.27)
+				)
+				(hide yes)
+			)
+		)
+		(property "Datasheet" ""
+			(at 41.91 44.45 0)
+			(effects
+				(font
+					(size 1.27 1.27)
+				)
+				(hide yes)
+			)
+		)
+		(property "Description" "Power symbol creates a global label with name \"+3.3V\""
+			(at 41.91 44.45 0)
+			(effects
+				(font
+					(size 1.27 1.27)
+				)
+				(hide yes)
+			)
+		)
+		(pin "1"
+		)
+		(instances
+			(project "VCU2.0"
+				(path "/3d82a156-9fcb-4cff-8c2b-14e72ba1cf3a/e5117eb9-18a3-4e8f-bd4d-5445d344d7ca"
+					(reference "#PWR0403")
+					(unit 1)
+				)
+			)
+		)
+	)
+	(symbol
 		(lib_id "ERJ3GEYJ100V:ERJ3GEYJ100V")
 		(at 166.37 46.99 270)
@@
 	)
 	(symbol
-		(lib_id "power:+5V")
-		(at 41.91 44.45 0)
+		(lib_id "power:+3.3V")
+		(at 90.17 26.67 0)
 		(unit 1)
 		(exclude_from_sim no)
@@
 		(dnp no)
 		(fields_autoplaced yes)
-		(property "Reference" "#PWR0403"
-			(at 41.91 48.26 0)
+		(property "Reference" "#PWR0401"
+			(at 90.17 30.48 0)
 			(effects
 				(font
@@
 			)
 		)
-		(property "Value" "+5V"
-			(at 41.91 39.37 0)
+		(property "Value" "+3.3V"
+			(at 90.17 21.59 0)
 			(effects
 				(font
@@
 		)
 		(property "Footprint" ""
-			(at 41.91 44.45 0)
+			(at 90.17 26.67 0)
 			(effects
 				(font
@@
 		)
 		(property "Datasheet" ""
-			(at 41.91 44.45 0)
+			(at 90.17 26.67 0)
 			(effects
 				(font
@@
 			)
 		)
-		(property "Description" "Power symbol creates a global label with name \"+5V\""
-			(at 41.91 44.45 0)
+		(property "Description" "Power symbol creates a global label with name \"+3.3V\""
+			(at 90.17 26.67 0)
 			(effects
 				(font
@@
 			(project "VCU2.0"
 				(path "/3d82a156-9fcb-4cff-8c2b-14e72ba1cf3a/e5117eb9-18a3-4e8f-bd4d-5445d344d7ca"
-					(reference "#PWR0403")
+					(reference "#PWR0401")
 					(unit 1)
 				)
@@
 					(unit 1)
 				)
-			)
-		)
-	)
-	(symbol
-		(lib_id "power:+5V")
-		(at 90.17 26.67 0)
-		(unit 1)
-		(exclude_from_sim no)
-		(in_bom yes)
-		(on_board yes)
-		(dnp no)
-		(fields_autoplaced yes)
-		(property "Reference" "#PWR0401"
-			(at 90.17 30.48 0)
-			(effects
-				(font
-					(size 1.27 1.27)
-				)
-				(hide yes)
-			)
-		)
-		(property "Value" "+5V"
-			(at 90.17 21.59 0)
-			(effects
-				(font
-					(size 1.27 1.27)
-				)
-			)
-		)
-		(property "Footprint" ""
-			(at 90.17 26.67 0)
-			(effects
-				(font
-					(size 1.27 1.27)
-				)
-				(hide yes)
-			)
-		)
-		(property "Datasheet" ""
-			(at 90.17 26.67 0)
-			(effects
-				(font
-					(size 1.27 1.27)
-				)
-				(hide yes)
-			)
-		)
-		(property "Description" "Power symbol creates a global label with name \"+5V\""
-			(at 90.17 26.67 0)
-			(effects
-				(font
-					(size 1.27 1.27)
-				)
-				(hide yes)
-			)
-		)
-		(pin "1"
-		)
-		(instances
-			(project "VCU2.0"
-				(path "/3d82a156-9fcb-4cff-8c2b-14e72ba1cf3a/e5117eb9-18a3-4e8f-bd4d-5445d344d7ca"
-					(reference "#PWR0401")
-					(unit 1)
-				)
