File: VCU2.0/Connector.kicad_sch (KiCad schematic)
At the start: 5 parts, among them U501 282815-3, U502 282815-3, U503 282815-3, U504 282815-3, U505 D-SUB-DR-25PCM-BB

Commit message: nice
Parts:
- added U506, U507: D-SUB-DR-9PCM-CB, footprint:DB9-TH_D-SUB-DR-9PCM-CB, symbol D-SUB-DR-9PCM-CB:D-SUB-DR-9PCM-CB
Connections:
- net CAN_H: now also U507.7
- net CAN_L: now also U507.2

Commit message: simple regen
Parts:
- added H501: 2x3, footprint:HDR-TH_6P-P2.54-V-M-R2-C3-S2.54-1, symbol Header-Male-2_54_2x3:Header-Male-2_54_2x3
Connections:
- net +3.3V: now also H501.2
- net CAN_H: now also U506.3
- net CAN_L: now also U506.5
- net GND: now also U506.10 (MH1), U506.11 (MH2), U507.10 (MH1), U507.11 (MH2), H501.6
- new net IO1: H501.1
- new net IO2: H501.3
- new net IO3: H501.5
- new net IO4: H501.4
Other:
- note added: "CAN IO"
- note added: "IO"
- moved on the sheet: U506, U507
