File: VCU2.0/Supply.kicad_sch (KiCad schematic)
At the start: 31 parts, among them U201 TPS564257DRLR, U202 TPS564257DRLR, U203 ADP3338AKC-3_3-RL

Commit message: simple regen
Parts:
- removed C213, C214: 1uF, footprint:C0805, symbol CL21B105KBFNNNE:CL21B105KBFNNNE
- removed L202: 4.7uH, footprint:IND-SMD_L3.3-W3.0, symbol SCD03015T-4R7M-NA:SCD03015T-4R7M-NA
- removed U203: ADP3338AKC-3_3-RL, footprint:SOT-223-3_L6.5-W3.4-P2.30-LS7.0-BR-1, symbol ADP3338AKC-3_3-RL:ADP3338AKC-3_3-RL
- added U203: SLO0530H4R7MTT, footprint:IND-SMD_L5.4-W5.2, symbol SLO0530H4R7MTT:SLO0530H4R7MTT
Connections:
- net +5V: now also U203.2
- net at U202.2 (SW): now also U203.1
Other:
- note removed: "BYPASS 3V3 (USB)"
