File: VCU2.0/VCU2.0.kicad_pcb (KiCad board)
At the start: 4 copper layers, 137.2 x 61.6 mm, 94 parts, among them IC601 TPS1HA08CQPWPRQ1, IC602 BTS716GB, IC603 BTS716GB, IC604 TPS1HA08CQPWPRQ1, SW301 Tactile, SW302 Tactile, U201 TPS564257DRLR, U202 TPS564257DRLR, U203 ADP3338AKC-3_3-RL, U301 ESP32-S3-WROOM-1(N8R2)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

Commit message: simple regen
Parts:
- removed C213, C214: 1uF, footprint:C0805
- removed H301: 2x3, footprint:HDR-TH_6P-P2.54-V-M-R2-C3-S2.54-1
- removed IC601, IC604: TPS1HA08CQPWPRQ1, footprint:SOP65P640X120-17N
- removed L202: 4.7uH, footprint:IND-SMD_L3.3-W3.0
- removed R601, R602, R603, R604: 2.7k, footprint:R0603
- removed SW301, SW302: Tactile, footprint:SW-SMD_4P-L6.0-W6.0-P4.50-LS9.0-2
- added H302: 2x3, footprint:HDR-TH_6P-P2.54-V-M-R2-C3-S2.54-1, F.Cu at (41.4, 137.9)
- added H501: 2x3, footprint:HDR-TH_6P-P2.54-V-M-R2-C3-S2.54-1, F.Cu at (63.8, 138.9)
- added U306: TS35CA, footprint:KEY-SMD_TS35CA, F.Cu at (47.5, 108.7)
- added U307: TS35CA, footprint:KEY-SMD_TS35CA, F.Cu at (53.8, 108.7)
- added U506: D-SUB-DR-9PCM-CB, footprint:DB9-TH_D-SUB-DR-9PCM-CB, F.Cu at (100.0, 116.3)
- added U507: D-SUB-DR-9PCM-CB, footprint:DB9-TH_D-SUB-DR-9PCM-CB, F.Cu at (135.0, 116.2)
- added U601: TC4429COA, footprint:SOIC-8_L4.9-W3.9-P1.27-LS6.0-BL, F.Cu at (143.8, 142.7)
- added U602: TC4429COA, footprint:SOIC-8_L4.9-W3.9-P1.27-LS6.0-BL, F.Cu at (137.2, 142.7)
- added U603: VBQA4317, footprint:PDFN-8_L5.9-W5.2-P1.27-LS6.2-BL-1, F.Cu at (147.1, 154.4)
- U203: value ADP3338AKC-3_3-RL -> SLO0530H4R7MTT; footprint footprint:SOT-223-3_L6.5-W3.4-P2.30-LS7.0-BR-1 -> footprint:IND-SMD_L5.4-W5.2
- moved U304 72.4 mm to (44.5, 119.4)
- moved C305 68.6 mm to (33.5, 120.8)
- moved R308 68.6 mm to (34.9, 117.0)
- moved U303 68.6 mm to (38.0, 124.0)
- moved C304 68.6 mm to (34.9, 118.8)
- moved R307 68.6 mm to (40.5, 117.6)
- moved U305 68.6 mm to (37.8, 111.9)
- moved U203 68.6 mm to (155.2, 131.1)
- moved R306 68.5 mm to (44.3, 124.5)
- moved R305 68.4 mm to (44.5, 122.4)
- moved U302 65.9 mm to (47.8, 120.1)
- moved R202 24.7 mm to (113.5, 124.0), turned to 90 degrees
- moved C203 24.3 mm to (113.5, 127.1), turned to -90 degrees
- moved R203 23.4 mm to (114.8, 131.6), turned to 0 degrees
- moved R205 22.8 mm to (114.8, 129.7), turned to 180 degrees
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Connections:
- net /IO/CAN_CS renamed /e/CAN_CS
- net /IO/CAN_IN renamed /e/CAN_IN
- net /IO/MISO renamed /e/MISO
- net /IO/MOSI renamed /e/MOSI
- net /IO/P1 renamed /e/P1
- net /IO/P2 renamed /e/P2
- net /IO/P3 renamed /e/P3
- net /IO/P4 renamed /e/P4
- net /IO/P5 renamed /e/P5
- net /IO/P6 renamed /e/P6
- net /IO/P7 renamed /e/P7
- net /IO/RXCAN renamed /e/RXCAN
- net /IO/SCK renamed /e/SCK
- net /IO/TXCAN renamed /e/TXCAN
- R401 pad 2: +5V -> +3.3V
- R402 pad 2: +5V -> +3.3V
- U203 pad 1: GND -> Net-(U202-SW)
- U203 pad 2: +3.3V -> +5V
- U301 pad 13: unconnected-(U301-IO19-Pad13) -> /Connector/IO2
- U301 pad 14: unconnected-(U301-IO20-Pad14) -> /Connector/IO1
- U301 pad 15: unconnected-(U301-IO3-Pad15) -> /Connector/IO3
- U301 pad 16: unconnected-(U301-IO46-Pad16) -> /Connector/IO4
- U301 pad 8: unconnected-(U301-IO15-Pad8) -> /esp32S3/EXT_CS
- U402 pad 20: +5V -> +3.3V
Routing:
- net /Connector/CAN_H: track 14.2 -> 150.3 mm, vias 0 -> 1
- net /Connector/CAN_L: track 11.4 -> 146.5 mm, vias 0 -> 1
- net /esp32S3/EN: track 104.8 -> 28.6 mm, vias 1 -> 0
- net /esp32S3/BOOT: track 112.3 -> 60.5 mm, vias 3 -> 2
- net Net-(IC601-DIA_EN): track 44.6 -> 0.00 mm
- net /PowerMGMT/PWI1: track 102.5 -> 62.7 mm
- net Net-(IC604-DIA_EN): track 39.7 -> 0.00 mm, vias 2 -> 0
- net /Connector/PWO0: track 39.1 -> 0.00 mm, vias 2 -> 0
- net /Connector/PWO1: track 32.3 -> 0.19 mm, vias 2 -> 0
- net /esp32S3/EXT_CS: track 0.00 -> 28.6 mm, vias 0 -> 2
- net /e/MOSI: track 29.9 -> 52.9 mm
- net VBUS: track 42.3 -> 20.1 mm, vias 1 -> 2
- net /e/MISO: track 29.0 -> 50.7 mm, vias 2 -> 0
- net /PowerMGMT/PWI0: track 90.5 -> 68.9 mm
- net Net-(U603A-G1): track 0.00 -> 20.4 mm
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- added copper zone on F.Cu, net /Connector/PWO0
- added copper zone on F.Cu, net /Connector/PWO1
Other:
- board text added: "BMS CAN"
- board text added: "PEAK CAN"
