File: VCU2.0/esp32S3.kicad_sch (KiCad schematic)
At the start: 21 parts, among them SW301 Tactile, SW302 Tactile, U301 ESP32-S3-WROOM-1(N8R2), U302 BC817, U303 CP2102N-A02-GQFN28R, U304 BC817, U305 YTC-TC16S-24

Commit message: simple regen
Parts:
- removed H301: 2x3, footprint:HDR-TH_6P-P2.54-V-M-R2-C3-S2.54-1, symbol Header-Male-2_54_2x3:Header-Male-2_54_2x3
- removed SW301, SW302: Tactile, footprint:SW-SMD_4P-L6.0-W6.0-P4.50-LS9.0-2, symbol KH-6X6X5H-STM:KH-6X6X5H-STM
- added H302: 2x3, footprint:HDR-TH_6P-P2.54-V-M-R2-C3-S2.54-1, symbol Header-Male-2_54_2x3:Header-Male-2_54_2x3
- added U306, U307: TS35CA, footprint:KEY-SMD_TS35CA, symbol TS35CA:TS35CA
Connections:
- net +3.3V: now also H302.2
- net BOOT: now also U306.2
- net EN: now also U307.2
- net GND: now also H302.6, U306.1, U306.3, U306.4, U307.1, U307.3, U307.4
- net MISO: now also H302.3
- net MOSI: now also H302.5
- net SCK: now also H302.1
- net IO1: now reaches U301.13 (IO19)
- net IO2: now reaches U301.14 (IO20)
- net IO3: now reaches U301.15 (IO3)
- net IO4: now reaches U301.16 (IO46)
- net EXT_CS: now reaches U301.8 (IO15)
- net EXT_CS: now also H302.4
- no-connect marks 27 -> 24
Other:
- note added: "SPI CON"
